File: atividades/atividade-03/vin-5v-regulator.brd (EAGLE design)
At the start: 160 x 100 mm, 10 parts, among them IC3 LM317

Commit message: roteamento automatico
Parts:
- moved R14 22.5 mm to (22.5, 4.57)
- moved R15 15.5 mm to (22.9, 8.89)
- moved C3 14.0 mm to (10.2, 21.6), turned to 180 degrees
- moved IC3 11.7 mm to (33.0, 33.0)
- moved D1 10.9 mm to (33.0, 52.1), turned to 90 degrees
- moved LED2 10.5 mm to (10.2, 31.8)
- moved R2 9.16 mm to (22.9, 14.0), turned to 180 degrees
- moved C4 4.02 mm to (22.9, 33.0), turned to 180 degrees
- moved C5 2.54 mm to (11.4, 44.5)
Routing:
- net GND: track 0.00 -> 106.3 mm
- net +5V: track 0.00 -> 55.5 mm
- net N$2: track 0.00 -> 30.3 mm
- net N$3: track 0.00 -> 29.3 mm
- net N$4: track 0.00 -> 24.6 mm
- net N$1: track 0.00 -> 18.4 mm
